Commit message: feat: replace urdf

File: xlerobot_pinc_urdf/robot.urdf (robot description, URDF)
Before this commit: robot robot, 15 links, 14 joints
Links:
- removed link cam
- removed link distal_shell
- removed link distal_shell_2
- removed link external_rod
- removed link external_rod_2
- removed link gripper_frame_link
- removed link internal_rod
- removed link internal_rod_2
- added link gripper_interface_link, mass 1e-09
- link interface_arm100: geometry 
Joints:
- removed joint Revolute 14
- removed joint Revolute 15
- removed joint Revolute 16
- removed joint Revolute 7
- removed joint Revolute 8
- removed joint Revolute 9
- removed joint gripper
- removed joint gripper_frame_fixed_joint
- added joint gripper_interface: type fixed, parent gripper_interface_link, child interface_arm100, origin xyz=0.0 0.0 0.0 rpy=0 3.14159 0
- joint elbow_flex: origin xyz=-0.112485 -0.028 0.0016 rpy=-4.39313e-16 1.9016e-16 1.5708 -> xyz=-0.112485 -0.028 0.0016 rpy=0.0 0.0 1.5708
- joint elbow_roll: origin xyz=-0.0626 3.33067e-16 0.0201 rpy=-1.5708 -2.80973e-14 -1.5708 -> xyz=-0.0626 0.0 0.0201 rpy=-1.5708 0.0 -1.5708
- joint shoulder_pan: origin xyz=0.0449 -0.000250002 0.0663 rpy=3.14159 1.07987e-08 3.14159 -> xyz=0.0449 -0.000250002 0.0663 rpy=3.14159 0.0 3.14159
- joint wrist_flex: origin xyz=-0.00498613 0.0198678 -0.0728416 rpy=1.5708 6.37128e-14 -4.4409e-16 -> xyz=-0.00498613 0.0198678 -0.0728416 rpy=1.5708 0.0 0.0
- joint wrist_roll: child interface_arm100 -> gripper_interface_link; origin xyz=-2.77556e-17 -0.0626 0.0201 rpy=1.5708 -1.10148e-13 3.14159 -> xyz=0.0 -0.0626 0.0201 rpy=1.5708 0.0 3.14159

Commit message: fix: add gripper_frame_link

File: xlerobot_pinc_urdf/robot.urdf (robot description, URDF)
Before this commit: robot robot, 8 links, 7 joints
Links:
- removed link interface_arm100
- added link gripper_frame_link, mass 1e-09
Joints:
- joint gripper_interface: child interface_arm100 -> gripper_frame_link; origin xyz=0.0 0.0 0.0 rpy=0 3.14159 0 -> xyz=0 0 -0.123609 rpy=0 1.5708 0
