Commit message: fix(gripper.urdf): make gripper base link name match the arm tcp name, i.e. rename gripper to cam

File: xlerobot_pinc_urdf/gripper.urdf (robot description, URDF)
Before this commit: robot gripper, 10 links, 9 joints
Joints:
- joint gripper_frame_fixed_joint: parent gripper -> cam

Commit message: feat: update urdf for so107_xl

File: xlerobot_pinc_urdf/gripper.urdf (robot description, URDF)
Before this commit: robot gripper, 10 links, 9 joints
Links:
- removed link tcp_link
- added link gripper_frame_link, mass 1e-9
- link interface_arm100: geometry collision mesh filename=package://assets/bottom_plate.stl; collision mesh filename=package://assets/camera_basement.stl
Joints:
- joint Revolute 16: origin xyz=0.034641 0.02 -0.008 rpy=1.11022e-15 -1.1989e-23 0.441689 -> xyz=0.034641 0.02 -0.008 rpy=-1.82922e-15 -1.15261e-15 0.441689
- joint Revolute 9: origin xyz=0.034641 0.02 -0.008 rpy=-3.14159 5.60794e-17 0.751294 -> xyz=0.034641 0.02 -0.008 rpy=3.14159 2.54324e-17 0.751294
- joint gripper: limit lower=-3.141592653589793 upper=3.141592653589793 effort=10 velocity=2 -> lower=-3.141592653589793 upper=3.141592653589793 effort=10 velocity=10; origin xyz=0.0029 1.4962e-17 -0.0455626 rpy=0 1.5708 0 -> xyz=0.0029 9.45424e-17 -0.0455626 rpy=6.12323e-17 1.5708 0
- joint gripper_frame_fixed_joint: child tcp_link -> gripper_frame_link; origin xyz=0.0 0.0 0.123609 rpy=0 0 0 -> xyz=-3.94522e-17 0 -0.123609 rpy=6.12323e-17 1.5708 0; parent cam -> interface_arm100

File: xlerobot_pinc_urdf/robot.urdf (robot description, URDF)
Before this commit: robot robot, 8 links, 7 joints
Links:
- removed link gripper_interface_link
- removed link upper_arm_so101_v1
- added link interface_arm100, mass 1e-09
- added link upper_arm_xl, mass 1e-09; collision mesh filename=package://assets/sts3215_03a_v1__3.stl; collision mesh filename=package://assets/upper_arm_xl.stl
- link gripper_frame_link: mass 1e-09 -> 1e-9
Joints:
- removed joint gripper_interface
- added joint gripper_frame_fixed_joint: type fixed, parent interface_arm100, child gripper_frame_link, origin xyz=-3.94522e-17 0 -0.123609 rpy=6.12323e-17 1.5708 0, axis 0 0 0
- joint elbow_flex: limit lower=-1.6580627893946132 upper=1.5707963267948966 effort=10 velocity=2 -> lower=-1.6580627893946132 upper=1.5707963267948966 effort=10 velocity=10; origin xyz=-0.112485 -0.028 0.0016 rpy=0.0 0.0 1.5708 -> xyz=-0.187485 -0.028 0.0016 rpy=-1.5234e-15 -1.37129e-14 1.5708; parent upper_arm_so101_v1 -> upper_arm_xl
- joint elbow_roll: origin xyz=-0.0626 0.0 0.0201 rpy=-1.5708 0.0 -1.5708 -> xyz=-0.0626 1.05626e-16 0.0201 rpy=-1.5708 -9.25644e-14 -1.5708
- joint shoulder_lift: child upper_arm_so101_v1 -> upper_arm_xl
- joint shoulder_pan: origin xyz=0.0449 -0.000250002 0.0663 rpy=3.14159 0.0 3.14159 -> xyz=0.0449 -0.000250002 0.0663 rpy=3.14159 1.05335e-08 3.12052
- joint wrist_flex: limit lower=-1.6580627893946132 upper=1.6580627893946132 effort=10 velocity=2 -> lower=-1.6580627893946132 upper=1.6580627893946132 effort=10 velocity=10; origin xyz=-0.00498613 0.0198678 -0.0728416 rpy=1.5708 0.0 0.0 -> xyz=0.0 0.0198678 -0.147842 rpy=1.5708 2.87986e-14 -2.22048e-16
- joint wrist_roll: child gripper_interface_link -> interface_arm100; origin xyz=0.0 -0.0626 0.0201 rpy=1.5708 0.0 3.14159 -> xyz=-8.18725e-17 -0.0626 0.0201 rpy=1.5708 -1.4468e-13 3.14159
